File: hardware_design/pcb/Voicecard-SMRMU-v01.brd (EAGLE design)
At the start: 118.7 x 60.3 mm, 117 parts, among them IC1 4052D, IC2 LM13700M, IC3 LM13700M, IC4 LM13700M, IC5 TL072, Q1 2N3906, Q2 2N3906, Q3 2N3906, Q4 2N3906, Q5 20MHz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

Commit message: Add boardlayout, assemblyfiles for v01 and pdf
Parts:
- removed U$6: (no value), og-pcb-art:V2_LOGO_SMALL
- added C17, C34, C35, C36, C37: 100n, jhbruhn-cdr:C0603
- added R56, R57, R58, R59, R60, R61, R62: 100k, jhbruhn-cdr:R0603
- Q6, Q7: value (none) -> 2N7002
- R18: value 160k -> 180k
- R20: value 330k -> 390k
- R44, R45, R51: value 49k9 -> 100k
- R47, R48: value 33k2 -> 100k
- moved JP5 142.4 mm to (3.17, 43.8), turned to 270 degrees
- moved R55 133.2 mm to (5.71, 40.0), turned to 270 degrees
- moved C31 123.2 mm to (104.8, 34.9), turned to 270 degrees
- moved R41 119.3 mm to (102.2, 34.9), turned to 270 degrees
- moved R53 119.0 mm to (64.8, 10.8)
- moved R54 117.5 mm to (64.8, 5.08)
- moved Q6 111.2 mm to (67.3, 8.89), turned to 90 degrees
- moved Q7 111.2 mm to (67.3, 3.17), turned to 90 degrees
- moved R52 94.4 mm to (50.8, 14.0), turned to 90 degrees
- moved R51 89.8 mm to (48.3, 14.0), turned to 90 degrees
- moved C33 86.7 mm to (43.8, 1.91), turned to 270 degrees
- moved R45 85.8 mm to (64.8, 14.0), turned to 90 degrees
- moved C32 85.1 mm to (46.4, 1.91), turned to 270 degrees
- moved R50 83.7 mm to (43.2, 14.0), turned to 90 degrees
- moved R44 81.5 mm to (62.2, 14.0), turned to 90 degrees
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Connections:
- net +5V: now also C35.1
- net 2P: now also R57.2, R61.2, R62.2
- net 3P: now also R56.2, R58.2, R59.2, R60.2
- net BP4: now also R56.1
- net GND: now also C17.2, C34.1, C35.2, C36.2, C37.1, IC4.13; no longer IC4.14
- net HP3: now also R59.1, R60.1, R61.1, R62.1
- net N$34: now also IC4.14; no longer IC4.13
- net NO: now also R57.1, R58.1
- net VCC: now also C17.1, C36.1
- net VEE: now also C34.2, C37.2
Routing:
- net 4P: track 28.4 -> 156.1 mm, vias 2 -> 19
- net N$15: track 0.00 -> 79.5 mm, vias 0 -> 8
- net VCC: track 161.3 -> 239.0 mm, vias 0 -> 10
- net 3P: track 27.3 -> 102.1 mm, vias 0 -> 12
- net N$11: track 5.10 -> 78.9 mm, vias 0 -> 2
- net 2P: track 61.9 -> 134.4 mm, vias 6 -> 16
- net N$20: track 4.71 -> 74.2 mm, vias 0 -> 2
- net N$10: track 70.5 -> 7.92 mm, vias 2 -> 0
- net N$7: track 69.5 -> 7.92 mm, vias 2 -> 0
- net CAPIN: track 10.5 -> 70.0 mm, vias 0 -> 10
- net 1P: track 41.3 -> 94.4 mm, vias 2 -> 8
- net VEE: track 236.8 -> 283.4 mm, vias 6 -> 14
- net PRE: track 0.00 -> 39.3 mm, vias 0 -> 4
- net MUXTB: track 0.00 -> 34.4 mm
- net VCA: track 51.4 -> 82.8 mm, vias 4 -> 6
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Other:
- board text added: "FM"
- board text added: "SMR-4MU voicecard"
- board text added: "v0.1"
- board text added: "Émilie Gillet, jhbruhn"
- board text removed: "Mutable Instruments"
- board text removed: "SMR-4 voicecard"
- board text removed: "v0.4smd"
- board text removed: "Émilie Gillet, SMD jhbruhn"
