File: hardware_design/pcb/Voicecard-SMRMU-v01.sch (EAGLE design)
At the start: 112 parts, among them IC1 4052D, IC2 LM13700M, IC3 LM13700M, IC4 LM13700M, IC5 TL072, Q1 2N3906, Q2 2N3906, Q3 2N3906, Q4 2N3906, Q5 20MHz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

Commit message: Add boardlayout, assemblyfiles for v01 and pdf
Parts:
- added C17, C34, C35, C36, C37: 100n, jhbruhn-cdr:C-EUC0603
- added R56, R57, R58, R59, R60, R61, R62: 100k, jhbruhn-cdr:R-EU_R0603
- Q6, Q7: value (none) -> 2N7002
- R18: value 160k -> 180k
- R20: value 330k -> 390k
- R44, R45, R51: value 49k9 -> 100k
- R47, R48: value 33k2 -> 100k
Connections:
- net +5V: now also C35.1
- net 2P: now also R57.2, R61.2, R62.2
- net 3P: now also R56.2, R58.2, R59.2, R60.2
- net BP4: now also R56.1
- net GND: now also C17.2, C34.1, C35.2, C36.2, C37.1, IC1P.GND, IC4OTA2.IN_N; no longer IC4OTA2.IN_P
- net HP3: now also R59.1, R60.1, R61.1, R62.1
- net N$34: now also IC4OTA2.IN_P; no longer IC4OTA2.IN_N
- net NO: now also R57.1, R58.1
- net VCC: now also C17.1, C36.1, IC1P.VCC
- net VEE: now also C34.2, C37.2, IC1P.VEE
Other:
- moved on the sheet: C1, C11, C13, C16, C18, C19, C20, C23, C24, C25, C28, C29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
