File: hardware_design/pcb/Voicecard-SMRMU-v02.sch (EAGLE design)
At the start: 125 parts, among them IC1 TL072CD, IC2 TL072CD, IC3 LM13700M, IC4 LM13700M, IC5 TL072, IC6 LM13700M, IC7 4052D, Q1 2N3906, Q2 2N3906, Q3 2N3906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

Commit message: Fix Multiplexer BOM Entry to use proper CMOS variant
Parts:
- IC7: value 4052D -> CD4052B; device jhbruhn-ic:4052D -> jhbruhn-ic:CD4052B
Changed lines of the file:
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@@
 <part name="C6" library="jhbruhn-cdr" deviceset="C-EU" device="C0603" package3d_urn="urn:adsk.eagle:package:23616/2" value="100n"/>
 <part name="C18" library="jhbruhn-cdr" deviceset="C-EU" device="C0603" package3d_urn="urn:adsk.eagle:package:23616/2" value="100n"/>
-<part name="IC7" library="jhbruhn-ic" deviceset="4052" device="D"/>
+<part name="IC7" library="jhbruhn-ic" deviceset="CD4052" device="B"/>
 <part name="R31" library="jhbruhn-cdr" deviceset="R-EU_" device="R0603" package3d_urn="urn:adsk.eagle:package:23555/42" value="22k"/>
 <part name="C22" library="jhbruhn-cdr" deviceset="C-EU" device="C0603" package3d_urn="urn:adsk.eagle:package:23616/2" value="10p"/>
